File: PCIe.kicad_sch (KiCad schematic)
At the start: 24 parts, among them J12 10018783-11200TLF, U15 AP64501SP-13

Commit message: Add files via upload
Parts:
- removed C25, C26, C27, C28, C43, C44: 10u 35v, Capacitor_SMD:C_0805_2012Metric, symbol Device:C
- removed C29, C62: 100n, Capacitor_SMD:C_0402_1005Metric, symbol Device:C
- removed C30, C31, C32, C33: 10u, Capacitor_SMD:C_0805_2012Metric, symbol Device:C
- removed C45: 100uF, Capacitor_Tantalum_SMD:CP_EIA-7343-31_Kemet-D, symbol Device:CP
- removed C63, C65: nf, Capacitor_SMD:C_0402_1005Metric, symbol Device:C
- removed C64: 1.2nF, Capacitor_SMD:C_0402_1005Metric, symbol Device:C
- removed J12: 10018783-11200TLF, CM4IO:PCIex1-36, symbol CM4IO:PCIe-x1
- removed L3: SRN6045TA-3R3Y, Inductor_SMD:L_Bourns_SRN6045TA, symbol pspice:INDUCTOR
- removed R22: 10R, Resistor_SMD:R_0402_1005Metric, symbol Device:R
- removed R23: 12K 1%, Resistor_SMD:R_0402_1005Metric, symbol Device:R
- removed R24: 47K 1%, Resistor_SMD:R_0402_1005Metric, symbol Device:R
- removed R30: 15K 1%, Resistor_SMD:R_0402_1005Metric, symbol Device:R
- removed TP1: TestPoint, TestPoint:TestPoint_Pad_2.0x2.0mm, symbol Connector:TestPoint
- removed U15: AP64501SP-13, CM4IO:SOIC-8-1EP_3.9x4.9mm_P1.27mm_EP2.95x4.9mm_Mask2.71x3.4mm_ThermalVias, symbol CM4IO:AP64351
Connections:
- no-connect marks 6 -> 0
Other:
- note removed: "3.3v @ 3.3A PSU for PCIe Only ( 12v Input )"
- note removed: "NB PCIe x1 takes a maximum of +12v @0.6A or +3.3v@3A , 10Watts combined"
- note removed: "PCIe x1 connector"
- note removed: "TX and RX have PN swaps to improve routing"
